File: Quantu_PiezoDriver-legacy/Quantu_PiezoDriver-legacy.kicad_pcb (KiCad board)
At the start: 2 copper layers, 102 x 100 mm, 115 parts, among them IC1 AD8221ARMZ, IC2 AD8221ARMZ, IC3 AD8671ARMZ-REEL, IC4 AD8671ARMZ-REEL, IC5 OPA445AU, IC6 UA79M05CKCS, IC7 AD8671ARMZ-REEL, IC8 AD8221ARMZ, IC9 AD8221ARMZ, J1 Ramp Voltage, J11 Conn_01x03, J2 Dither Voltage, J3 HV Output, J4 LV Monitor, J5 Feed Forward, J7 Conn_02x02_Odd_Even, SW1 SW_SPST, SW2 SW_SPST, SW3 SW_SPST, U1 LM399, U2 AD8606ARZ

Commit message: replace potentiometer footprint for Bourns 3339H
Parts:
- RV1, RV3: footprint Potentiometer_THT:Potentiometer_Bourns_3296Y_Vertical -> Potentiometer_THT:Potentiometer_Bourns_3339H_Vertical
- RV2: footprint Potentiometer_THT:Potentiometer_Bourns_3296W_Vertical -> Potentiometer_THT:Potentiometer_Bourns_3339H_Vertical
- moved RV1 4.44 mm to (12.0, 37.4), turned to 90 degrees
- moved RV2 2.65 mm to (76.1, 29.6), turned to -90 degrees
- moved RV3 0.58 mm to (90.6, 58.3), turned to 90 degrees
Routing:
- net GND: track 40.9 -> 24.2 mm
- net Net-(PS1-VADJ._1): track 7.41 -> 12.9 mm
- net VS: track 112.0 -> 117.1 mm
- net Net-(PS1-V_REF_1): track 7.43 -> 11.6 mm
- net Net-(IC3-+IN): track 14.0 -> 14.8 mm
- net Net-(U2B--): track 13.7 -> 13.0 mm
