File: Quantu_PiezoDriver-legacy/Quantu_PiezoDriver-legacy.kicad_sch (KiCad schematic)
At the start: 115 parts, among them IC1 AD8221ARMZ, IC2 AD8221ARMZ, IC3 AD8671ARMZ-REEL, IC4 AD8671ARMZ-REEL, IC5 OPA445AU, IC6 UA79M05CKCS, IC7 AD8671ARMZ-REEL, IC8 AD8221ARMZ, IC9 AD8221ARMZ, J1 Ramp Voltage, J11 Conn_01x03, J2 Dither Voltage, J3 HV Output, J4 LV Monitor, J5 Feed Forward, J7 Conn_02x02_Odd_Even, SW1 SW_SPST, SW2 SW_SPST, SW3 SW_SPST, U1 LM399, U2 AD8606ARZ

Commit message: replace potentiometer footprint for Bourns 3339H
Parts:
- RV1, RV3: footprint Potentiometer_THT:Potentiometer_Bourns_3296Y_Vertical -> Potentiometer_THT:Potentiometer_Bourns_3339H_Vertical
- RV2: footprint Potentiometer_THT:Potentiometer_Bourns_3296W_Vertical -> Potentiometer_THT:Potentiometer_Bourns_3339H_Vertical
Changed lines of the file:
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@@
 			)
 		)
-		(property "Footprint" "Potentiometer_THT:Potentiometer_Bourns_3296Y_Vertical"
+		(property "Footprint" "Potentiometer_THT:Potentiometer_Bourns_3339H_Vertical"
 			(at 81.28 189.23 0)
 			(effects
@@
 			)
 		)
-		(property "Footprint" "Potentiometer_THT:Potentiometer_Bourns_3296Y_Vertical"
+		(property "Footprint" "Potentiometer_THT:Potentiometer_Bourns_3339H_Vertical"
 			(at 119.38 97.79 0)
 			(effects
@@
 			)
 		)
-		(property "Footprint" "Potentiometer_THT:Potentiometer_Bourns_3296W_Vertical"
+		(property "Footprint" "Potentiometer_THT:Potentiometer_Bourns_3339H_Vertical"
 			(at 219.71 35.56 0)
 			(effects
